Commit message: initial

File: src/process_visualizer/urdf/arm_basis1.urdf (robot description, URDF)
Before this commit: robot arm_basis, 2 links, 1 joints
Links:
- link arm_basis: geometry visual mesh filename=package://process_visualizer/resources/arm_basis1.STL

File: src/process_visualizer/urdf/box_ur5.xacro (robot description, xacro)
@@ -32,5 +32,5 @@
     </gazebo>
     <gazebo reference="object_link">
-        <material>Gazebo/Blue</material>
+        <material>Gazebo/Turquoise</material>
     </gazebo>
 </robot>

File: src/universal_robot/ur_description/urdf/ur5.urdf.xacro (robot description, xacro)
@@ -101,7 +101,7 @@
       <axis xyz="0 0 1" />
       <xacro:unless value="${joint_limited}">
-        <limit lower="${-2.0 * pi}" upper="${2.0 * pi}" effort="150.0" velocity="3.15"/>
-        <xacro:if value="${safety_limits}">
-          <safety_controller soft_lower_limit="${-2.0 * pi + safety_pos_margin}" soft_upper_limit="${2.0 * pi - safety_pos_margin}" k_position="${safety_k_position}" k_velocity="0.0"/>
+        <limit lower="${-pi}" upper="${pi}" effort="150.0" velocity="3.15"/>
+        <xacro:if value="${safety_limits}">
+          <safety_controller soft_lower_limit="${-pi + safety_pos_margin}" soft_upper_limit="${pi - safety_pos_margin}" k_position="${safety_k_position}" k_velocity="0.0"/>
         </xacro:if>
       </xacro:unless>
@@ -138,7 +138,7 @@
       <axis xyz="0 1 0" />
       <xacro:unless value="${joint_limited}">
-        <limit lower="${-2.0 * pi}" upper="${2.0 * pi}" effort="150.0" velocity="3.15"/>
-        <xacro:if value="${safety_limits}">
-          <safety_controller soft_lower_limit="${-2.0 * pi + safety_pos_margin}" soft_upper_limit="${2.0 * pi - safety_pos_margin}" k_position="${safety_k_position}" k_velocity="0.0"/>
+        <limit lower="${-pi}" upper="${pi}" effort="150.0" velocity="3.15"/>
+        <xacro:if value="${safety_limits}">
+          <safety_controller soft_lower_limit="${-pi + safety_pos_margin}" soft_upper_limit="${pi - safety_pos_margin}" k_position="${safety_k_position}" k_velocity="0.0"/>
         </xacro:if>
       </xacro:unless>
@@ -177,5 +177,5 @@
         <limit lower="${-pi}" upper="${pi}" effort="150.0" velocity="3.15"/>
         <xacro:if value="${safety_limits}">
-          <safety_controller soft_lower_limit="${-2.0 * pi + safety_pos_margin}" soft_upper_limit="${2.0 * pi - safety_pos_margin}" k_position="${safety_k_position}" k_velocity="0.0"/>
+          <safety_controller soft_lower_limit="${-pi + safety_pos_margin}" soft_upper_limit="${pi - safety_pos_margin}" k_position="${safety_k_position}" k_velocity="0.0"/>
         </xacro:if>
       </xacro:unless>
@@ -212,7 +212,7 @@
       <axis xyz="0 1 0" />
       <xacro:unless value="${joint_limited}">
-        <limit lower="${-2.0 * pi}" upper="${2.0 * pi}" effort="28.0" velocity="3.2"/>
-        <xacro:if value="${safety_limits}">
-          <safety_controller soft_lower_limit="${-2.0 * pi + safety_pos_margin}" soft_upper_limit="${2.0 * pi - safety_pos_margin}" k_position="${safety_k_position}" k_velocity="0.0"/>
+        <limit lower="${-pi}" upper="${pi}" effort="28.0" velocity="3.2"/>
+        <xacro:if value="${safety_limits}">
+          <safety_controller soft_lower_limit="${-pi + safety_pos_margin}" soft_upper_limit="${pi - safety_pos_margin}" k_position="${safety_k_position}" k_velocity="0.0"/>
         </xacro:if>
       </xacro:unless>
@@ -249,7 +249,7 @@
       <axis xyz="0 0 1" />
       <xacro:unless value="${joint_limited}">
-        <limit lower="${-2.0 * pi}" upper="${2.0 * pi}" effort="28.0" velocity="3.2"/>
-        <xacro:if value="${safety_limits}">
-          <safety_controller soft_lower_limit="${-2.0 * pi + safety_pos_margin}" soft_upper_limit="${2.0 * pi - safety_pos_margin}" k_position="${safety_k_position}" k_velocity="0.0"/>
+        <limit lower="${-pi}" upper="${pi}" effort="28.0" velocity="3.2"/>
+        <xacro:if value="${safety_limits}">
+          <safety_controller soft_lower_limit="${-pi + safety_pos_margin}" soft_upper_limit="${pi - safety_pos_margin}" k_position="${safety_k_position}" k_velocity="0.0"/>
         </xacro:if>
       </xacro:unless>
@@ -286,7 +286,7 @@
       <axis xyz="0 1 0" />
       <xacro:unless value="${joint_limited}">
-        <limit lower="${-2.0 * pi}" upper="${2.0 * pi}" effort="28.0" velocity="3.2"/>
-        <xacro:if value="${safety_limits}">
-          <safety_controller soft_lower_limit="${-2.0 * pi + safety_pos_margin}" soft_upper_limit="${2.0 * pi - safety_pos_margin}" k_position="${safety_k_position}" k_velocity="0.0"/>
+        <limit lower="${-pi}" upper="${pi}" effort="28.0" velocity="3.2"/>
+        <xacro:if value="${safety_limits}">
+          <safety_controller soft_lower_limit="${-pi + safety_pos_margin}" soft_upper_limit="${pi - safety_pos_margin}" k_position="${safety_k_position}" k_velocity="0.0"/>
         </xacro:if>
       </xacro:unless>
